File: SIx5-7-x/TW5-x-7.kicad_sch (KiCad schematic)
At the start: 4 parts

Commit message: テンプレを作成↓
Parts:
- H1, H2, H3, H4: footprint MountingHole:MountingHole_2.7mm -> MountingHole:MountingHole_2.2mm_M2
Changed lines of the file:
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@@
       (effects (font (size 1.27 1.27)) (justify left))
     )
-    (property "Footprint" "MountingHole:MountingHole_2.7mm" (at 21.8694 177.7746 0)
+    (property "Footprint" "MountingHole:MountingHole_2.2mm_M2" (at 21.8694 177.7746 0)
       (effects (font (size 1.27 1.27)) hide)
     )
@@
     )
     (instances
-      (project "SIx5-7-x"
+      (project "TW5-x-7"
         (path "/b4c24110-5ce2-4b9b-89f1-7a788ee960b8"
           (reference "H1") (unit 1)
@@
       (effects (font (size 1.27 1.27)) (justify left))
     )
-    (property "Footprint" "MountingHole:MountingHole_2.7mm" (at 44.3484 178.1556 0)
+    (property "Footprint" "MountingHole:MountingHole_2.2mm_M2" (at 44.3484 178.1556 0)
       (effects (font (size 1.27 1.27)) hide)
     )
@@
     )
     (instances
-      (project "SIx5-7-x"
+      (project "TW5-x-7"
         (path "/b4c24110-5ce2-4b9b-89f1-7a788ee960b8"
           (reference "H3") (unit 1)
@@
       (effects (font (size 1.27 1.27)) (justify left))
     )
-    (property "Footprint" "MountingHole:MountingHole_2.7mm" (at 44.3484 186.2836 0)
+    (property "Footprint" "MountingHole:MountingHole_2.2mm_M2" (at 44.3484 186.2836 0)
       (effects (font (size 1.27 1.27)) hide)
     )
@@
     )
     (instances
-      (project "SIx5-7-x"
+      (project "TW5-x-7"
         (path "/b4c24110-5ce2-4b9b-89f1-7a788ee960b8"
           (reference "H4") (unit 1)
@@
       (effects (font (size 1.27 1.27)) (justify left))
     )
-    (property "Footprint" "MountingHole:MountingHole_2.7mm" (at 21.8694 186.563 0)
+    (property "Footprint" "MountingHole:MountingHole_2.2mm_M2" (at 21.8694 186.563 0)
       (effects (font (size 1.27 1.27)) hide)
     )
@@
     )
     (instances
-      (project "SIx5-7-x"
+      (project "TW5-x-7"
         (path "/b4c24110-5ce2-4b9b-89f1-7a788ee960b8"
           (reference "H2") (unit 1)
